File: swweeep/choc-hotswap-optional/half-swept.kicad_pcb (KiCad board)
At the start: 2 copper layers, 113.3 x 89.7 mm, 34 parts, among them J1 JST-BATTERY, SW1 SW_Push, SW10 SW_Push, SW11 SW_Push, SW12 SW_Push, SW14 SW_Push, SW15 SW_Push, SW16 SW_Push, SW17 SW_Push, SW18 SW_Push, SW2 SW_Push, SW20 SW_Push, SW21 SW_Push, SW3 SW_Push, SW4 SW_Push, SW5 SW_Push, SW6 SW_Push, SW7 SW_DPDT, SW8 SW_Push, SW9 SW_Push, U1 nice_nano

Commit message: Swweep34
Parts:
- removed SW1: SW_Push, fingerpunch:Kailh_socket_PG1350_optional_reversible_millmax
- moved SW21 8.77 mm to (86.3, 82.3)
- moved SW20 8.46 mm to (104.9, 90.0), turned to 150 degrees
Connections:
- U1 pad 20: Switch18 -> unconnected-(U1-AIN7/P0.31-Pad20)
Routing:
- net Switch18: track 99.2 -> 0.00 mm, vias 2 -> 0
- net gnd: track 31.6 -> 94.2 mm, vias 4 -> 5
- net Switch17: track 76.7 -> 86.3 mm
- net Switch16: track 66.5 -> 72.4 mm
