File: swweeep/choc-hotswap-optional/half-swept.kicad_sch (KiCad schematic)
At the start: 31 parts, among them J1 JST-BATTERY, SW1 SW_Push, SW10 SW_Push, SW11 SW_Push, SW12 SW_Push, SW14 SW_Push, SW15 SW_Push, SW16 SW_Push, SW17 SW_Push, SW18 SW_Push, SW2 SW_Push, SW20 SW_Push, SW21 SW_Push, SW3 SW_Push, SW4 SW_Push, SW5 SW_Push, SW6 SW_Push, SW7 SW_DPDT, SW8 SW_Push, SW9 SW_Push, U1 nice_nano

Commit message: Swweep34
Parts:
- removed SW1: SW_Push, fingerpunch:Kailh_socket_PG1350_optional_reversible_millmax, symbol Switch:SW_Push
Connections:
- net Switch18: no longer names the net of U1.20 (AIN7/P0.31)
- no-connect marks 0 -> 1
